File: UccMicroDuino/_autosave-UccMicroDuino.kicad_pcb (KiCad board)
At the start: 2 copper layers, 51.9 x 45 mm, 14 parts, among them J1 pcb USB type A, J2 HEADER, U1 ATtiny85-20S

Commit message: Add files via upload
Parts:
- moved J2 146.9 mm to (265.5, 92.1), turned to 180 degrees
- moved U1 139.0 mm to (265.6, 63.1), turned to 180 degrees
- moved C1 114.6 mm to (250.6, 91.7)
- moved D2 108.1 mm to (235.3, 69.7)
- moved D1 101.1 mm to (224.8, 63.9), turned to 180 degrees
- moved J1 96.8 mm to (224.0, 56.0), turned to -90 degrees
- moved R1 95.4 mm to (233.6, 63.9), turned to 180 degrees
- moved D3 88.7 mm to (223.8, 76.8), turned to 180 degrees
- moved D4 85.0 mm to (235.8, 84.2)
- moved R3 83.7 mm to (229.2, 76.8)
- moved D5 82.2 mm to (232.9, 92.1)
- moved R5 81.5 mm to (226.7, 92.1)
- moved R2 79.4 mm to (224.6, 69.4)
- moved R4 79.3 mm to (224.8, 84.2)
